Commit message: 修复navigation2无法导航问题

File: src/kamibot_base/description/kamibot.xacro (robot description, xacro)
@@ -1,22 +1,22 @@
 <?xml version="1.0"?>
 <robot xmlns:xacro="http://www.ros.org/wiki/xacro" name="kamibot">
-    <xacro:include filename="kamibot_materials.xacro" />
     <xacro:property name="base_mass" value="1" />
     <xacro:property name="base_radius" value="0.20" />  <!-- 底盘半径 -->
     <xacro:property name="base_height" value="0.16" />  <!-- 底盘高度 -->
     <xacro:property name="wheel_mass" value="0.2" />
-    <xacro:property name="wheel_radius" value="0.06" />  <!-- 轮子半径 -->
-    <xacro:property name="wheel_length" value="0.025" /> <!-- 轮子厚度 -->
-    <xacro:property name="wheel_joint_y" value="0.19" />
-    <xacro:property name="wheel_joint_z" value="-0.05" />
-    <xacro:property name="caster_radius" value="0.015" />
-    <xacro:property name="caster_joint_x" value="0.17" />
-    <xacro:property name="caster_joint_z" value="-0.095" />
+    <xacro:property name="wheel_radius" value="0.04" />  <!-- 轮子半径 -->
+    <xacro:property name="wheel_length" value="0.02" /> <!-- 轮子厚度 -->
+    <xacro:property name="wheel_joint_y" value="${base_radius}" />
+    <xacro:property name="wheel_joint_z" value="${-base_height/2}" />
+    <xacro:property name="base_groud_height" value="${wheel_radius}" />  <!-- 底盘离地高度 -->
+    <xacro:property name="caster_radius" value="${wheel_radius/2}" />
+    <xacro:property name="caster_joint_x" value="${base_radius-caster_radius}" />
+    <xacro:property name="caster_joint_z" value="${-(base_height/2+caster_radius)}" />
     <xacro:property name="lidar_mass" value="0.1" />
-    <xacro:property name="lidar_radius" value="0.05" />
-    <xacro:property name="lidar_height" value="0.04" />
-    <xacro:property name="lidar_joint_x" value="0.15" />
-    <xacro:property name="lidar_joint_z" value="0.10" />
-    <xacro:property name="camera_joint_x" value="0.20" />
+    <xacro:property name="lidar_radius" value="${base_radius/4}" />
+    <xacro:property name="lidar_height" value="${base_height/4}" />
+    <xacro:property name="lidar_joint_x" value="${base_radius-lidar_radius}" />
+    <xacro:property name="lidar_joint_z" value="${base_height/2+lidar_height/2}" />
+    <xacro:property name="camera_joint_x" value="${base_radius}" />
     <!-- 生成底座 -->
     <xacro:include filename="kamibot_base.xacro" />
@@ -26,4 +26,5 @@
         r="${base_radius}"
         h="${base_height}"
+        g="${base_groud_height}"
         color="Gazebo/Turquoise"
     />
@@ -48,5 +49,5 @@
         name="front_caster"
         r="${caster_radius}"
-        color="Gazebo/RedGlow"
+        color="Gazebo/TurquoiseGlow"
     />
     <xacro:caster_macro
@@ -62,10 +63,12 @@
         r="${lidar_radius}"
         h="${lidar_height}"
-        color="Gazebo/DarkGrey"
+        color="Gazebo/RedGlow"
     />
     <!-- 生成相机 -->
     <xacro:include filename="sensors/camera_gazebo.xacro" />
-    <xacro:usb_camera name="kamibot_camera" />
-    <!-- 关节定义，连接以上组件 -->
+    <xacro:usb_camera
+        name="kamibot_camera"
+        color="Gazebo/RedGlow"
+    />
     <!-- 左轮关节 -->
     <joint name="left_wheel_joint" type="continuous">

File: src/kamibot_base/description/kamibot_base.xacro (robot description, xacro)
@@ -1,6 +1,23 @@
 <?xml version="1.0"?>
 <robot xmlns:xacro="http://www.ros.org/wiki/xacro">
+    <xacro:include filename="kamibot_utils.xacro" />
     <!-- 圆柱形底盘 -->
-    <xacro:macro name="base_macro" params="name m r h color">
+    <xacro:macro name="base_macro" params="name m r h g color">
+        <link name="base_footprint">
+            <visual>
+                <origin xyz="0 0 0" rpy="0 0 0" />
+                <geometry>
+                    <box size="0.001 0.001 0.001" />
+                </geometry>
+            </visual>
+        </link>
+        <gazebo reference="base_footprint">
+            <turnGravityOff>false</turnGravityOff>
+        </gazebo>
+        <joint name="base_footprint_joint" type="fixed">
+            <origin xyz="0 0 ${h/2+g}" rpy="0 0 0" />
+            <parent link="base_footprint"/>
+            <child link="${name}" />
+        </joint>
         <link name="${name}">
             <visual>
@@ -9,4 +26,7 @@
                     <cylinder length="${h}" radius="${r}"/>
                 </geometry>
+                <material name="green">
+                    <color rgba="0 0.5 0 1"/>
+                </material>
             </visual>
             <collision>
@@ -16,5 +36,4 @@
                 </geometry>
             </collision>
-            <xacro:include filename="kamibot_utils.xacro" />
             <xacro:cylinder_inertial_matrix m="${m}" r="${r}" h="${h}" />
         </link>

File: src/kamibot_base/description/kamibot_wheel.xacro (robot description, xacro)
@@ -1,4 +1,5 @@
 <?xml version="1.0"?>
 <robot xmlns:xacro="http://www.ros.org/wiki/xacro">
+    <xacro:include filename="kamibot_utils.xacro" />
     <!-- 驱动轮宏 -->
     <xacro:macro name="drive_wheel_macro" params="name m r h color">
@@ -8,5 +9,7 @@
                     <cylinder radius="${r}" length="${h}" />
                 </geometry>
-                <material name="yellow" />
+                <material name="black">
+                    <color rgba="0 0 0 1"/>
+                </material>
                 <origin rpy="${pi/2} 0 0" xyz="0 0 0" /> <!--旋转90度-->
             </visual>
@@ -17,5 +20,4 @@
                 <origin rpy="${pi/2} 0 0" xyz="0 0 0" />
             </collision>
-            <xacro:include filename="kamibot_utils.xacro" />
             <xacro:cylinder_inertial_matrix m="${m}" r="${r}" h="${h}" />
         </link>
@@ -42,12 +44,15 @@
     <xacro:macro name="caster_macro" params="name r color">
         <link name="${name}">
-            <xacro:include filename="kamibot_utils.xacro" />
             <visual>
+                <origin xyz="0 0 0" rpy="0 0 0"/>
                 <geometry>
                     <sphere radius="${r}" />
                 </geometry>
-                <material name="yellow" />
+                <material name="black">
+                    <color rgba="0 0 0 1"/>
+                </material>
             </visual>
             <collision>
+                <origin xyz="0 0 0" rpy="0 0 0"/>
                 <geometry>
                     <sphere radius="${r}" />

File: src/kamibot_base/description/sensors/camera_gazebo.xacro (robot description, xacro)
@@ -1,5 +1,5 @@
 <?xml version="1.0"?>
 <robot xmlns:xacro="http://www.ros.org/wiki/xacro" name="camera">
-    <xacro:macro name="usb_camera" params="name:=camera prefix:=kamibot">
+    <xacro:macro name="usb_camera" params="name:=camera prefix:=kamibot color">
         <link name="${name}">
             <inertial>
@@ -25,5 +25,5 @@
         </link>
         <gazebo reference="${name}">
-            <material>Gazebo/FlatBlack</material>
+            <material>color</material>
         </gazebo>
         <gazebo reference="${name}">

Commit message: 修改nav2巡航错误问题

File: src/kamibot_base/description/kamibot.xacro (robot description, xacro)
@@ -10,4 +10,5 @@
     <xacro:property name="wheel_joint_z" value="${-base_height/2}" />
     <xacro:property name="base_groud_height" value="${wheel_radius}" />  <!-- 底盘离地高度 -->
+    <xacro:property name="caster_mass" value="0.1" />
     <xacro:property name="caster_radius" value="${wheel_radius/2}" />
     <xacro:property name="caster_joint_x" value="${base_radius-caster_radius}" />
@@ -48,4 +49,5 @@
     <xacro:caster_macro
         name="front_caster"
+        m="${caster_mass}"
         r="${caster_radius}"
         color="Gazebo/TurquoiseGlow"
@@ -53,4 +55,5 @@
     <xacro:caster_macro
         name="back_caster"
+        m="${caster_mass}"
         r="${caster_radius}"
         color="Gazebo/TurquoiseGlow"

File: src/kamibot_base/description/kamibot_utils.xacro (robot description, xacro)
@@ -1,4 +1,12 @@
 <?xml version="1.0"?>
 <robot xmlns:xacro="http://www.ros.org/wiki/xacro">
+    <xacro:macro name="sphere_inertial_matrix" params="m r">
+        <inertial>
+            <mass value="${m}" />
+            <inertia ixx="${2*m*r*r/5}" ixy="0" ixz="0"
+                iyy="${2*m*r*r/5}" iyz="0"
+                izz="${2*m*r*r/5}" />
+        </inertial>
+    </xacro:macro>
     <xacro:macro name="cylinder_inertial_matrix" params="m r h">
         <inertial>

File: src/kamibot_base/description/kamibot_wheel.xacro (robot description, xacro)
@@ -42,5 +42,5 @@
     </xacro:macro>
     <!-- 万向轮宏 -->
-    <xacro:macro name="caster_macro" params="name r color">
+    <xacro:macro name="caster_macro" params="name m r color">
         <link name="${name}">
             <visual>
@@ -59,4 +59,5 @@
                 </geometry>
             </collision>
+            <xacro:sphere_inertial_matrix  m="${m}" r="${r}" />
         </link>
         <gazebo reference="${name}">

Commit message: 添加导航逻辑

File: src/kamibot_base/description/kamibot.xacro (robot description, xacro)
@@ -17,5 +17,4 @@
     <xacro:property name="lidar_radius" value="${base_radius/4}" />
     <xacro:property name="lidar_height" value="${base_height/4}" />
-    <xacro:property name="lidar_joint_x" value="${base_radius-lidar_radius}" />
     <xacro:property name="lidar_joint_z" value="${base_height/2+lidar_height/2}" />
     <xacro:property name="camera_joint_x" value="${base_radius}" />
@@ -106,5 +105,5 @@
         <parent link="base_link" />
         <child link="kamibot_lidar" />
-        <origin xyz="${lidar_joint_x} 0 ${lidar_joint_z}" />
+        <origin xyz="0 0 ${lidar_joint_z}" />
     </joint>
     <!-- 相机关节 -->
