Commit message: 格式化python代码

File: src/kamibot_base/description/sensors/camera_gazebo.xacro (robot description, xacro)
@@ -11,5 +11,5 @@
             </inertial>
             <visual>
-                <origin xyz=" 0 0 0 " rpy="0 0 0" />
+                <origin xyz=" 0 0 0 " rpy="${-1.57} 0 0" />
                 <geometry>
                     <box size="0.01 0.04 0.04" />
@@ -18,5 +18,5 @@
             </visual>
             <collision>
-                <origin xyz="0.0 0.0 0.0" rpy="0 0 0" />
+                <origin xyz="0.0 0.0 0.0" rpy="${-1.57} 0 0" />
                 <geometry>
                     <box size="0.01 0.04 0.04" />
@@ -26,4 +26,5 @@
         <gazebo reference="${name}">
             <material>color</material>
+            <origin xyz="0 0 0" rpy="${-1.57} 0 0" />
         </gazebo>
         <gazebo reference="${name}">
